Commit message: Organized moveit utilities a bit - now it is possible to plan for two arms from python interface

File: two_arms_ur_utilities/urdf/ur3_left_joint_limited_robot.urdf.xacro (robot description, xacro)
@@ -21,5 +21,5 @@
     <parent link="world" />
     <child link = "left_arm_base_link" />
-    <origin xyz="0.0 0.3 0.2" rpy="0.0 0.0 0.0" />
+    <origin xyz="0.0 0.4 0.6" rpy="0.0 0.0 0.0" />
   </joint>
 </robot>

File: two_arms_ur_utilities/urdf/ur3_left_robot.urdf.xacro (robot description, xacro)
@@ -15,5 +15,5 @@
     <parent link="world" />
     <child link = "left_arm_base_link" />
-    <origin xyz="0.0 0.3 0.2" rpy="0.0 0.0 0.0" />
+    <origin xyz="0.0 0.4 0.6" rpy="0.0 0.0 0.0" />
   </joint>
 </robot>

File: two_arms_ur_utilities/urdf/ur3_right_joint_limited_robot.urdf.xacro (robot description, xacro)
@@ -21,5 +21,5 @@
     <parent link="world" />
     <child link = "right_arm_base_link" />
-    <origin xyz="0.0 -0.3 0.2" rpy="0.0 0.0 0.0" />
+    <origin xyz="0.0 -0.4 0.6" rpy="0.0 0.0 0.0" />
   </joint>
 </robot>

File: two_arms_ur_utilities/urdf/ur3_right_robot.urdf.xacro (robot description, xacro)
@@ -15,5 +15,5 @@
     <parent link="world" />
     <child link = "right_arm_base_link" />
-    <origin xyz="0.0 -0.3 0.2" rpy="0.0 0.0 0.0" />
+    <origin xyz="0.0 -0.4 0.6" rpy="0.0 0.0 0.0" />
   </joint>
 </robot>
